File: skyshieldv0.2.brd (EAGLE design)
At the start: 17.8 x 43.2 mm, 17 parts, among them IC2 MCP1702-5, J1 HEAD15-NOSS, J2 HEAD15-NOSS-1

Commit message: update
Connections:
- removed net N$5: J2.12, JP2.1
- removed net VIN: IC2.2, J2.1, JP1.1
- new net A2: J2.10, RLED1.1
- new net N$6: IC2.2, JP1.1
- net A0: now also J2.12, JP2.1; no longer J2.11, RLED.1
- net A1: now also J2.11, RLED.1; no longer J2.10, RLED1.1
- net VCC: now also J2.1
Changed lines of the file:
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@@
 <wire x1="8.636" y1="5.842" x2="1.27" y2="19.0246" width="0" layer="19" extent="1-1"/>
-</signal>
-<signal name="A1">
-<contactref element="RLED1" pad="1"/>
-<contactref element="J2" pad="10"/>
-<wire x1="6.35" y1="13.4112" x2="1.27" y2="16.4846" width="0" layer="19" extent="1-1"/>
-</signal>
-<signal name="A0">
-<contactref element="RLED" pad="1"/>
-<contactref element="J2" pad="11"/>
-<wire x1="1.27" y1="13.9446" x2="4.064" y2="13.462" width="0" layer="19" extent="1-1"/>
 </signal>
 <signal name="A4">
@@
 <contactref element="RLED3" pad="1"/>
 <wire x1="11.4554" y1="1.9558" x2="1.27" y2="31.7246" width="0" layer="19" extent="1-1"/>
-</signal>
-<signal name="VIN">
-<contactref element="J2" pad="1"/>
-<contactref element="IC2" pad="2"/>
-<contactref element="JP1" pad="1"/>
-<wire x1="1.27" y1="39.3446" x2="7.6454" y2="40.8432" width="0" layer="19" extent="1-1"/>
-<wire x1="6.6294" y1="37.9476" x2="7.6454" y2="40.8432" width="0" layer="19" extent="1-1"/>
 </signal>
 <signal name="3V3">
@@
 <contactref element="SV4" pad="5"/>
 <contactref element="SV4" pad="2"/>
+<contactref element="J2" pad="1"/>
 <wire x1="12.4206" y1="36.0934" x2="11.2014" y2="40.9194" width="0" layer="19" extent="1-1"/>
 <wire x1="7.8994" y1="36.0426" x2="12.4206" y2="36.0934" width="0" layer="19" extent="1-1"/>
 <wire x1="12.3698" y1="30.4292" x2="12.4206" y2="36.0934" width="0" layer="19" extent="1-1"/>
+<wire x1="1.27" y1="39.3446" x2="7.8994" y2="36.0426" width="0" layer="19" extent="1-1"/>
 <wire x1="12.3698" y1="22.8092" x2="12.3698" y2="30.4292" width="0" layer="19" extent="1-1"/>
 <wire x1="12.3698" y1="15.1892" x2="12.3698" y2="22.8092" width="0" layer="19" extent="1-1"/>
@@
 <wire x1="4.064" y1="5.842" x2="8.4328" y2="31.4198" width="0" layer="19" extent="1-1"/>
 </signal>
-<signal name="N$5">
-<contactref element="J2" pad="12"/>
-<contactref element="JP2" pad="1"/>
-<wire x1="1.27" y1="11.4046" x2="4.2418" y2="17.7292" width="0" layer="19" extent="1-1"/>
-</signal>
 <signal name="N$4">
 <contactref element="SWITCH" pad="2"/>
@@
 <wire x1="13.7668" y1="9.5504" x2="11.4554" y2="9.5758" width="0" layer="19" extent="1-1"/>
 </signal>
+<signal name="N$6">
+<contactref element="IC2" pad="2"/>
+<contactref element="JP1" pad="1"/>
+<wire x1="6.6294" y1="37.9476" x2="7.6454" y2="40.8432" width="0" layer="19" extent="1-1"/>
+</signal>
+<signal name="A2">
+<contactref element="J2" pad="10"/>
+<contactref element="RLED1" pad="1"/>
+<wire x1="1.27" y1="16.4846" x2="6.35" y2="13.4112" width="0" layer="19" extent="1-1"/>
+</signal>
+<signal name="A1">
+<contactref element="J2" pad="11"/>
+<contactref element="RLED" pad="1"/>
+<wire x1="1.27" y1="13.9446" x2="4.064" y2="13.462" width="0" layer="19" extent="1-1"/>
+</signal>
+<signal name="A0">
+<contactref element="J2" pad="12"/>
+<contactref element="JP2" pad="1"/>
+<wire x1="1.27" y1="11.4046" x2="4.2418" y2="17.7292" width="0" layer="19" extent="1-1"/>
+</signal>
 </signals>

Commit message: update
Parts:
- removed JP2: USB, SparkFun:1X02_LOCK_LONGPADS
- removed RLED, RLED1, RLED2: 1.5K, rcl:0204/7
- removed SWITCH: adafruit, SparkFun:1X02_LOCK_LONGPADS
- added CHDK1A, CHDK1B, CHDK2A, CHDK2B, SW1A, SW1B: (no value), pinhead:1X01
- added R1, R2, R3: 1.5K, rcl:0204/7
- RS1: value 1.5K -> 100
- RS2: value 1.5K -> 10K
- moved JP1 0.69 mm to (8.20, 40.9)
- moved LED2 0.61 mm to (7.11, 22.8)
- moved LED1 0.59 mm to (7.11, 27.4)
- moved LED 0.51 mm to (7.14, 31.9)
- moved C4 0.20 mm to (12.7, 40.9)
- renumbered RLED3 to RS2, RLED4 to RS1
Connections:
- new net N$5: SW1A.1
- net A0: now also CHDK1A.1; no longer JP2.1
- net A1: now also CHDK2A.1; no longer RLED.1
- net A2: now also R1.1; no longer RLED1.1
- net A3: now also R2.1; no longer RLED2.1
- net A4: now also R3.1
- net GND: now also CHDK1B.1, CHDK2B.1, SW1B.1; no longer JP2.2, SWITCH.1
- net N$1: now also R3.2; no longer RLED2.2
- net N$2: now also R2.2; no longer RLED1.2
- net N$3: now also R1.2; no longer RLED.2
- net N$4: no longer SWITCH.2
Routing:
- removed copper zone on layer 1, net COM
- removed copper zone on layer 16, net COM
Other:
- outline, holes or cut-outs redrawn
- board text added: "R1"
- board text added: "R2"
- board text added: "R3"
- board text added: "RS1"
- board text added: "RS2"
- board text added: "S"
- board text added: "TX"
- board text added: "VIN"

Commit message: update
Parts:
- R1, R2, R3: value 1.5K -> 10K
- moved CHDK2B 3.78 mm to (7.49, 19.1)
- moved CHDK2A 3.73 mm to (4.90, 19.1)
- moved CHDK1A 3.66 mm to (4.93, 15.3)
- moved CHDK1B 3.66 mm to (7.49, 15.3)
Changed lines of the file:
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@@
 <wire x1="10.4902" y1="26.5938" x2="14.2748" y2="26.5938" width="0.4064" layer="21"/>
 <wire x1="10.5664" y1="18.9484" x2="14.351" y2="18.9484" width="0.4064" layer="21"/>
-<text x="4.5974" y="16.637" size="1.016" layer="21" ratio="15">-</text>
+<text x="4.4958" y="16.6624" size="1.016" layer="21" ratio="15">-</text>
 <text x="9.1948" y="18.669" size="0.8128" layer="21" ratio="15" rot="R270">CHDK</text>
-<text x="7.1882" y="16.637" size="1.016" layer="21" ratio="15">+</text>
-<text x="3.4798" y="19.431" size="1.016" layer="21" ratio="15" rot="R180">A</text>
-<text x="3.4544" y="15.9004" size="1.016" layer="21" ratio="15" rot="R180">B</text>
+<text x="7.0866" y="16.6624" size="1.016" layer="21" ratio="15">+</text>
+<text x="3.4544" y="15.8496" size="1.016" layer="21" ratio="15" rot="R180">A</text>
+<text x="3.4798" y="19.6342" size="1.016" layer="21" ratio="15" rot="R180">B</text>
 <text x="2.4892" y="1.5494" size="1.016" layer="21" ratio="15">S</text>
 <text x="4.4958" y="7.8994" size="1.016" layer="21" ratio="15" rot="R90">R1</text>
@@
 <element name="J1" library="MyCON2" package="HEAD15-NOSS" value="HEAD15-NOSS" x="16.4846" y="39.37" rot="R270"/>
 <element name="J2" library="MyCON2" package="HEAD15-NOSS-1" value="HEAD15-NOSS-1" x="1.27" y="39.3446" rot="R270"/>
-<element name="R1" library="rcl" package="0204/7" value="1.5K" x="3.8862" y="8.636" rot="R270"/>
+<element name="R1" library="rcl" package="0204/7" value="10K" x="3.8862" y="8.636" rot="R270"/>
 <element name="IC2" library="JeeLabs" package="TO92" value="MCP1702-5" x="6.6294" y="36.0426"/>
 <element name="C5" library="resistor" package="E1,8-4" value="10µ" x="12.4206" y="36.9824" rot="R90"/>
@@
 <attribute name="VALUE" x="15.2908" y="22.8092" size="1.27" layer="27" ratio="10" rot="R90"/>
 </element>
-<element name="R2" library="rcl" package="0204/7" value="1.5K" x="6.1976" y="8.636" rot="R270"/>
+<element name="R2" library="rcl" package="0204/7" value="10K" x="6.1976" y="8.636" rot="R270"/>
 <element name="LED1" library="adafruit" package="LED3MM" value="POWERLED" x="7.112" y="27.432" rot="R180"/>
-<element name="R3" library="rcl" package="0204/7" value="1.5K" x="8.5852" y="8.636" rot="R90"/>
+<element name="R3" library="rcl" package="0204/7" value="10K" x="8.5852" y="8.636" rot="R90"/>
 <element name="LED2" library="adafruit" package="LED3MM" value="POWERLED" x="7.112" y="22.8346" rot="R180"/>
 <element name="RS2" library="rcl" package="0204/7" value="10K" x="11.4554" y="5.7658" rot="R90"/>
 <element name="RS1" library="rcl" package="0204/7" value="100" x="13.7668" y="5.7404" rot="R270"/>
-<element name="CHDK1A" library="pinhead" package="1X01" value="" x="4.953" y="18.9484"/>
-<element name="CHDK1B" library="pinhead" package="1X01" value="" x="7.493" y="18.923"/>
-<element name="CHDK2A" library="pinhead" package="1X01" value="" x="4.9784" y="15.367"/>
-<element name="CHDK2B" library="pinhead" package="1X01" value="" x="7.5184" y="15.3162"/>
+<element name="CHDK1A" library="pinhead" package="1X01" value="" x="4.9276" y="15.2908"/>
+<element name="CHDK1B" library="pinhead" package="1X01" value="" x="7.493" y="15.2654"/>
+<element name="CHDK2A" library="pinhead" package="1X01" value="" x="4.9022" y="19.1008"/>
+<element name="CHDK2B" library="pinhead" package="1X01" value="" x="7.493" y="19.1008"/>
 <element name="SW1B" library="pinhead" package="1X01" value="" x="5.0038" y="2.1336"/>
 <element name="SW1A" library="pinhead" package="1X01" value="" x="7.5692" y="2.159"/>
@@
 <wire x1="5.842" y1="27.432" x2="5.8674" y2="31.9278" width="0" layer="19" extent="1-1"/>
 <wire x1="5.842" y1="22.8346" x2="5.842" y2="27.432" width="0" layer="19" extent="1-1"/>
-<wire x1="7.493" y1="18.923" x2="5.842" y2="22.8346" width="0" layer="19" extent="1-1"/>
-<wire x1="7.5184" y1="15.3162" x2="7.493" y2="18.923" width="0" layer="19" extent="1-1"/>
+<wire x1="7.493" y1="15.2654" x2="5.842" y2="22.8346" width="0" layer="19" extent="1-1"/>
+<wire x1="7.493" y1="19.1008" x2="7.493" y2="15.2654" width="0" layer="19" extent="1-1"/>
 <wire x1="5.5372" y1="40.8686" x2="5.3594" y2="36.0426" width="0" layer="19" extent="1-1"/>
-<wire x1="12.3698" y1="17.7292" x2="7.493" y2="18.923" width="0" layer="19" extent="1-1"/>
+<wire x1="12.3698" y1="17.7292" x2="7.493" y2="15.2654" width="0" layer="19" extent="1-1"/>
 <wire x1="12.3698" y1="25.3492" x2="5.842" y2="27.432" width="0" layer="19" extent="1-1"/>
-<wire x1="5.0038" y1="2.1336" x2="7.5184" y2="15.3162" width="0" layer="19" extent="1-1"/>
+<wire x1="5.0038" y1="2.1336" x2="7.493" y2="19.1008" width="0" layer="19" extent="1-1"/>
 </signal>
 <signal name="VCC" class="1">
@@
 <contactref element="J2" pad="11"/>
 <contactref element="CHDK2A" pad="1"/>
-<wire x1="1.27" y1="13.9446" x2="4.9784" y2="15.367" width="0" layer="19" extent="1-1"/>
+<wire x1="1.27" y1="13.9446" x2="4.9022" y2="19.1008" width="0" layer="19" extent="1-1"/>
 </signal>
 <signal name="A0">
 <contactref element="J2" pad="12"/>
 <contactref element="CHDK1A" pad="1"/>
-<wire x1="1.27" y1="11.4046" x2="4.953" y2="18.9484" width="0" layer="19" extent="1-1"/>
+<wire x1="1.27" y1="11.4046" x2="4.9276" y2="15.2908" width="0" layer="19" extent="1-1"/>
 </signal>
 <signal name="N$5">

Commit message: update
Parts:
- moved CHDK2B 0.72 mm to (6.99, 18.6)
- moved CHDK2A 0.68 mm to (4.45, 18.6)
- moved CHDK1B 0.64 mm to (6.96, 14.9)
- moved CHDK1A 0.64 mm to (4.42, 14.9)
- moved RS1 0.46 mm to (13.8, 6.20)
- moved RS2 0.38 mm to (11.5, 6.15)
- moved SW1A 0.28 mm to (7.57, 1.88)
- moved SW1B 0.25 mm to (5.00, 1.88)
Other:
- board text added: "CM1"
- board text added: "CM2"
- board text added: "D12"
- board text removed: "CHDK"
Changed lines of the file:
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@@
 <wire x1="10.4902" y1="26.5938" x2="14.2748" y2="26.5938" width="0.4064" layer="21"/>
 <wire x1="10.5664" y1="18.9484" x2="14.351" y2="18.9484" width="0.4064" layer="21"/>
-<text x="4.4958" y="16.6624" size="1.016" layer="21" ratio="15">-</text>
-<text x="9.1948" y="18.669" size="0.8128" layer="21" ratio="15" rot="R270">CHDK</text>
-<text x="7.0866" y="16.6624" size="1.016" layer="21" ratio="15">+</text>
-<text x="3.4544" y="15.8496" size="1.016" layer="21" ratio="15" rot="R180">A</text>
-<text x="3.4798" y="19.6342" size="1.016" layer="21" ratio="15" rot="R180">B</text>
-<text x="2.4892" y="1.5494" size="1.016" layer="21" ratio="15">S</text>
+<text x="4.0386" y="16.2306" size="1.016" layer="21" ratio="15">-</text>
+<text x="6.6294" y="16.1798" size="1.016" layer="21" ratio="15">+</text>
+<text x="8.8646" y="16.383" size="1.016" layer="21" ratio="15" rot="R270">CM1</text>
+<text x="8.8646" y="19.939" size="1.016" layer="21" ratio="15" rot="R270">CM2</text>
+<text x="9.271" y="1.397" size="1.016" layer="21" ratio="15">S</text>
 <text x="4.4958" y="7.8994" size="1.016" layer="21" ratio="15" rot="R90">R1</text>
 <text x="6.6802" y="7.874" size="1.016" layer="21" ratio="15" rot="R90">R2</text>
 <text x="9.0932" y="7.8994" size="1.016" layer="21" ratio="15" rot="R90">R3</text>
-<text x="14.2494" y="4.6736" size="1.016" layer="21" ratio="15" rot="R90">RS1</text>
-<text x="11.938" y="4.6482" size="1.016" layer="21" ratio="15" rot="R90">RS2</text>
+<text x="14.3002" y="4.9784" size="1.016" layer="21" ratio="15" rot="R90">RS1</text>
+<text x="11.9634" y="4.9276" size="1.016" layer="21" ratio="15" rot="R90">RS2</text>
 <wire x1="0" y1="40.7162" x2="2.4892" y2="43.18" width="0" layer="20" curve="-94.264616"/>
 <wire x1="15.3162" y1="43.18" x2="17.78" y2="40.6908" width="0" layer="20" curve="-94.264616"/>
@@
 <text x="10.5156" y="43.0784" size="1.016" layer="21" ratio="15" rot="R180">+</text>
 <text x="3.4036" y="42.1386" size="1.016" layer="21" ratio="15">-</text>
+<text x="16.4592" y="2.9718" size="1.016" layer="21" ratio="15" rot="R225">D12</text>
 </plain>
 <attributes>
@@
 <element name="R3" library="rcl" package="0204/7" value="10K" x="8.5852" y="8.636" rot="R90"/>
 <element name="LED2" library="adafruit" package="LED3MM" value="POWERLED" x="7.112" y="22.8346" rot="R180"/>
-<element name="RS2" library="rcl" package="0204/7" value="10K" x="11.4554" y="5.7658" rot="R90"/>
-<element name="RS1" library="rcl" package="0204/7" value="100" x="13.7668" y="5.7404" rot="R270"/>
-<element name="CHDK1A" library="pinhead" package="1X01" value="" x="4.9276" y="15.2908"/>
-<element name="CHDK1B" library="pinhead" package="1X01" value="" x="7.493" y="15.2654"/>
-<element name="CHDK2A" library="pinhead" package="1X01" value="" x="4.9022" y="19.1008"/>
-<element name="CHDK2B" library="pinhead" package="1X01" value="" x="7.493" y="19.1008"/>
-<element name="SW1B" library="pinhead" package="1X01" value="" x="5.0038" y="2.1336"/>
-<element name="SW1A" library="pinhead" package="1X01" value="" x="7.5692" y="2.159"/>
+<element name="RS2" library="rcl" package="0204/7" value="10K" x="11.4808" y="6.1468" rot="R90"/>
+<element name="RS1" library="rcl" package="0204/7" value="100" x="13.843" y="6.1976" rot="R270"/>
+<element name="CHDK1A" library="pinhead" package="1X01" value="" x="4.4196" y="14.9098"/>
+<element name="CHDK1B" library="pinhead" package="1X01" value="" x="6.9596" y="14.9098"/>
+<element name="CHDK2A" library="pinhead" package="1X01" value="" x="4.445" y="18.5928"/>
+<element name="CHDK2B" library="pinhead" package="1X01" value="" x="6.985" y="18.5928"/>
+<element name="SW1B" library="pinhead" package="1X01" value="" x="5.0038" y="1.8796"/>
+<element name="SW1A" library="pinhead" package="1X01" value="" x="7.5692" y="1.8796"/>
 </elements>
 <signals>
@@
 <contactref element="J1" pad="15"/>
 <contactref element="RS1" pad="2"/>
-<wire x1="13.7668" y1="1.9304" x2="16.4846" y2="3.81" width="0" layer="19" extent="1-1"/>
+<wire x1="13.843" y1="2.3876" x2="16.4846" y2="3.81" width="0" layer="19" extent="1-1"/>
 </signal>
 <signal name="A3">
@@
 <contactref element="J2" pad="4"/>
 <contactref element="RS2" pad="1"/>
-<wire x1="11.4554" y1="1.9558" x2="1.27" y2="31.7246" width="0" layer="19" extent="1-1"/>
+<wire x1="11.4808" y1="2.3368" x2="1.27" y2="31.7246" width="0" layer="19" extent="1-1"/>
 </signal>
 <signal name="3V3">
@@
 <wire x1="5.842" y1="27.432" x2="5.8674" y2="31.9278" width="0" layer="19" extent="1-1"/>
 <wire x1="5.842" y1="22.8346" x2="5.842" y2="27.432" width="0" layer="19" extent="1-1"/>
-<wire x1="7.493" y1="15.2654" x2="5.842" y2="22.8346" width="0" layer="19" extent="1-1"/>
-<wire x1="7.493" y1="19.1008" x2="7.493" y2="15.2654" width="0" layer="19" extent="1-1"/>
+<wire x1="6.9596" y1="14.9098" x2="5.842" y2="22.8346" width="0" layer="19" extent="1-1"/>
+<wire x1="6.985" y1="18.5928" x2="6.9596" y2="14.9098" width="0" layer="19" extent="1-1"/>
 <wire x1="5.5372" y1="40.8686" x2="5.3594" y2="36.0426" width="0" layer="19" extent="1-1"/>
-<wire x1="12.3698" y1="17.7292" x2="7.493" y2="15.2654" width="0" layer="19" extent="1-1"/>
+<wire x1="12.3698" y1="17.7292" x2="6.9596" y2="14.9098" width="0" layer="19" extent="1-1"/>
 <wire x1="12.3698" y1="25.3492" x2="5.842" y2="27.432" width="0" layer="19" extent="1-1"/>
-<wire x1="5.0038" y1="2.1336" x2="7.493" y2="19.1008" width="0" layer="19" extent="1-1"/>
+<wire x1="5.0038" y1="1.8796" x2="6.985" y2="18.5928" width="0" layer="19" extent="1-1"/>
 </signal>
 <signal name="VCC" class="1">
@@
 <contactref element="RS2" pad="2"/>
 <contactref element="RS1" pad="1"/>
-<wire x1="11.4554" y1="9.5758" x2="13.7668" y2="9.5504" width="0" layer="19" extent="1-1"/>
+<wire x1="11.4808" y1="9.9568" x2="13.843" y2="10.0076" width="0" layer="19" extent="1-1"/>
 </signal>
 <signal name="N$6">
@@
 <contactref element="J2" pad="11"/>
 <contactref element="CHDK2A" pad="1"/>
-<wire x1="1.27" y1="13.9446" x2="4.9022" y2="19.1008" width="0" layer="19" extent="1-1"/>
+<wire x1="1.27" y1="13.9446" x2="4.445" y2="18.5928" width="0" layer="19" extent="1-1"/>
 </signal>
 <signal name="A0">
 <contactref element="J2" pad="12"/>
 <contactref element="CHDK1A" pad="1"/>
-<wire x1="1.27" y1="11.4046" x2="4.9276" y2="15.2908" width="0" layer="19" extent="1-1"/>
+<wire x1="1.27" y1="11.4046" x2="4.4196" y2="14.9098" width="0" layer="19" extent="1-1"/>
 </signal>
 <signal name="N$5">
