File: skyshieldv0.3.brd (EAGLE design)
At the start: 17.8 x 43.2 mm, 21 parts, among them IC1 LD117AV, J1 HEAD15-NOSS, J2 HEAD15-NOSS-1

Commit message: update
Parts:
- moved C2 0.82 mm to (12.6, 40.9)
- moved C1 0.36 mm to (14.3, 36.5)
Routing:
- net VCC: track 47.9 -> 52.1 mm, vias 1 -> 0
- net GND: track 88.1 -> 87.3 mm
Changed lines of the file:
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@@
 <attribute name="VALUE" x="3.7592" y="17.3736" size="0.9906" layer="27" ratio="10" rot="R270"/>
 </element>
-<element name="C2" library="resistor" package="E1,8-4" value="10µ" x="12.573" y="41.6814" smashed="yes" rot="R180">
-<attribute name="VALUE" x="10.414" y="43.4594" size="1.27" layer="27" ratio="10" rot="R180"/>
-</element>
-<element name="C1" library="resistor" package="C025-024X044" value="0.1µ" x="14.3002" y="36.8808" smashed="yes" rot="R90">
-<attribute name="VALUE" x="16.9672" y="35.1028" size="1.27" layer="27" ratio="10" rot="R90"/>
+<element name="C2" library="resistor" package="E1,8-4" value="10µ" x="12.6492" y="40.8686" smashed="yes" rot="R180">
+<attribute name="VALUE" x="10.4902" y="42.6466" size="1.27" layer="27" ratio="10" rot="R180"/>
+</element>
+<element name="C1" library="resistor" package="C025-024X044" value="0.1µ" x="14.2748" y="36.5252" smashed="yes" rot="R90">
+<attribute name="VALUE" x="16.9418" y="34.7472" size="1.27" layer="27" ratio="10" rot="R90"/>
 </element>
 <element name="JP1" library="SparkFun" package="1X02_LOCK_LONGPADS" value="BATT" x="8.0772" y="41.148" smashed="yes" rot="R180">
@@
 <contactref element="J2" pad="3"/>
 <contactref element="J1" pad="3"/>
-<wire x1="11.5824" y1="34.29" x2="1.3716" y2="34.29" width="0.4064" layer="1"/>
-<wire x1="11.7348" y1="34.1376" x2="11.5824" y2="34.29" width="0.4064" layer="1"/>
-<wire x1="16.3068" y1="34.1376" x2="11.7348" y2="34.1376" width="0.4064" layer="1"/>
+<wire x1="13.716" y1="34.29" x2="1.3716" y2="34.29" width="0.4064" layer="1"/>
+<wire x1="13.8684" y1="34.1376" x2="13.716" y2="34.29" width="0.4064" layer="1"/>
+<wire x1="16.3068" y1="34.1376" x2="13.8684" y2="34.1376" width="0.4064" layer="1"/>
 <wire x1="16.4592" y1="34.29" x2="16.3068" y2="34.1376" width="0.4064" layer="1"/>
 <wire x1="1.3716" y1="34.29" x2="1.27" y2="34.2646" width="0.4064" layer="1"/>
@@
 <contactref element="SW1B" pad="1"/>
 <contactref element="IC1" pad="1"/>
-<wire x1="11.7348" y1="40.6908" x2="11.7348" y2="41.6052" width="0.8128" layer="16"/>
-<wire x1="14.1732" y1="38.2524" x2="11.7348" y2="40.6908" width="0.8128" layer="16"/>
-<wire x1="11.7348" y1="41.6052" x2="11.684" y2="41.6814" width="0.8128" layer="16"/>
-<wire x1="14.1732" y1="38.2524" x2="14.3002" y2="38.1508" width="0.8128" layer="16"/>
+<wire x1="11.8872" y1="40.0812" x2="11.8872" y2="40.8432" width="0.8128" layer="16"/>
+<wire x1="14.1732" y1="37.7952" x2="11.8872" y2="40.0812" width="0.8128" layer="16"/>
+<wire x1="11.8872" y1="40.8432" x2="11.7602" y2="40.8686" width="0.8128" layer="16"/>
+<wire x1="14.1732" y1="37.7952" x2="14.2748" y2="37.7952" width="0.8128" layer="16"/>
 <wire x1="13.5636" y1="26.5176" x2="12.4968" y2="25.4508" width="0.8128" layer="16"/>
 <wire x1="13.716" y1="26.5176" x2="13.5636" y2="26.5176" width="0.8128" layer="16"/>
@@
 <wire x1="15.3162" y1="30.5562" x2="12.954" y2="32.9184" width="0.8128" layer="16"/>
 <wire x1="12.4968" y1="32.9184" x2="12.3698" y2="32.9692" width="0.8128" layer="16"/>
-<wire x1="14.1732" y1="37.338" x2="14.1732" y2="37.7952" width="0.8128" layer="16"/>
-<wire x1="12.954" y1="36.1188" x2="14.1732" y2="37.338" width="0.8128" layer="16"/>
-<wire x1="12.954" y1="33.2232" x2="12.954" y2="36.1188" width="0.8128" layer="16"/>
-<wire x1="14.1732" y1="37.7952" x2="14.3002" y2="38.1508" width="0.8128" layer="16"/>
+<wire x1="14.0208" y1="36.7284" x2="14.0208" y2="37.4904" width="0.8128" layer="16"/>
+<wire x1="12.954" y1="35.6616" x2="14.0208" y2="36.7284" width="0.8128" layer="16"/>
+<wire x1="12.954" y1="33.2232" x2="12.954" y2="35.6616" width="0.8128" layer="16"/>
+<wire x1="14.0208" y1="37.4904" x2="14.2748" y2="37.7952" width="0.8128" layer="16"/>
 <wire x1="12.954" y1="33.2232" x2="12.3698" y2="32.9692" width="0.8128" layer="16"/>
 <wire x1="1.3716" y1="36.7284" x2="5.4864" y2="36.7284" width="0.8128" layer="1"/>
@@
 <wire x1="12.4968" y1="15.24" x2="12.3698" y2="15.1892" width="0.8128" layer="1"/>
 <wire x1="12.4968" y1="22.86" x2="12.3698" y2="22.8092" width="0.8128" layer="1"/>
-<wire x1="13.4112" y1="39.0144" x2="13.4112" y2="41.6052" width="0.8128" layer="1"/>
-<wire x1="12.954" y1="38.5572" x2="13.4112" y2="39.0144" width="0.8128" layer="1"/>
-<wire x1="12.954" y1="36.8808" x2="12.954" y2="38.5572" width="0.8128" layer="1"/>
-<wire x1="14.1732" y1="35.6616" x2="13.335" y2="36.4998" width="0.8128" layer="1"/>
-<wire x1="13.335" y1="36.4998" x2="12.954" y2="36.8808" width="0.8128" layer="1"/>
-<wire x1="13.4112" y1="41.6052" x2="13.462" y2="41.6814" width="0.8128" layer="1"/>
-<wire x1="14.1732" y1="35.6616" x2="14.3002" y2="35.6108" width="0.8128" layer="1"/>
+<wire x1="13.4112" y1="38.7096" x2="13.4112" y2="40.8432" width="0.8128" layer="1"/>
+<wire x1="12.954" y1="38.2524" x2="13.4112" y2="38.7096" width="0.8128" layer="1"/>
+<wire x1="12.954" y1="36.576" x2="12.954" y2="38.2524" width="0.8128" layer="1"/>
+<wire x1="14.2748" y1="35.2552" x2="12.954" y2="36.576" width="0.8128" layer="1"/>
+<wire x1="13.4112" y1="40.8432" x2="13.5382" y2="40.8686" width="0.8128" layer="1"/>
 <wire x1="12.0396" y1="30.48" x2="12.3444" y2="30.48" width="0.8128" layer="16"/>
-<wire x1="8.0772" y1="34.4424" x2="9.525" y2="32.9946" width="0.8128" layer="16"/>
-<wire x1="9.525" y1="32.9946" x2="12.0396" y2="30.48" width="0.8128" layer="16"/>
+<wire x1="8.0772" y1="34.4424" x2="12.0396" y2="30.48" width="0.8128" layer="16"/>
 <wire x1="8.0772" y1="36.576" x2="8.0772" y2="34.4424" width="0.8128" layer="16"/>
 <wire x1="12.3444" y1="30.48" x2="12.3698" y2="30.4292" width="0.8128" layer="16"/>
@@
 <wire x1="1.3716" y1="39.3192" x2="1.27" y2="39.3446" width="0.8128" layer="16"/>
 <wire x1="8.0772" y1="36.8808" x2="8.0264" y2="36.6268" width="0.8128" layer="16"/>
-<wire x1="11.8872" y1="35.052" x2="13.335" y2="36.4998" width="0.8128" layer="1"/>
-<wire x1="11.2776" y1="34.4424" x2="11.8872" y2="35.052" width="0.8128" layer="16"/>
-<wire x1="10.9728" y1="34.4424" x2="11.2776" y2="34.4424" width="0.8128" layer="16"/>
-<wire x1="9.525" y1="32.9946" x2="10.9728" y2="34.4424" width="0.8128" layer="16"/>
+<wire x1="12.3444" y1="42.0624" x2="13.5382" y2="40.8686" width="0.8128" layer="16"/>
+<wire x1="11.1252" y1="42.0624" x2="12.3444" y2="42.0624" width="0.8128" layer="16"/>
+<wire x1="9.6012" y1="40.5384" x2="11.1252" y2="42.0624" width="0.8128" layer="16"/>
+<wire x1="9.6012" y1="39.7764" x2="9.6012" y2="40.5384" width="0.8128" layer="16"/>
+<wire x1="7.62" y1="37.7952" x2="9.6012" y2="39.7764" width="0.8128" layer="16"/>
+<wire x1="7.62" y1="37.7952" x2="8.0264" y2="36.6268" width="0.8128" layer="16"/>
 <wire x1="13.5636" y1="23.9268" x2="12.8016" y2="23.1648" width="0.8128" layer="1"/>
 <wire x1="13.716" y1="23.9268" x2="13.5636" y2="23.9268" width="0.8128" layer="1"/>
@@
 <wire x1="12.8016" y1="23.1648" x2="12.3698" y2="22.8092" width="0.8128" layer="1"/>
 <wire x1="12.4968" y1="30.48" x2="12.3698" y2="30.4292" width="0.8128" layer="1"/>
-<via x="11.8872" y="35.052" extent="1-16" drill="0.3302"/>
 </signal>
 <signal name="D8">
