File: skyshieldv0.4.brd (EAGLE design)
At the start: 17.8 x 43.2 mm, 18 parts, among them J1 HEAD15-NOSS, J2 HEAD15-NOSS-1

Commit message: update
Parts:
- moved BATT 0.27 mm to (4.45, 40.6)
Routing:
- net A4: track 13.1 -> 13.8 mm
Other:
- board text added: ".com"
- board text added: "SKY-SWEEP"
- board text added: "v0.4"
- board text removed: "sky-sweep"
- board text removed: "ver0.3"
